File: analysis/Scenario2.sch (KiCad schematic (older format))
At the start: 6 parts, among them Q1 BS170

Commit message: add 2.png
Parts:
- removed L1: 55mH, symbol Device:L
- removed R3: 33, symbol Device:R
Connections:
- net +12V: now also D1.2 (A), Q1.1 (D)
Other:
- note removed: "Solenoid"
Changed lines of the file:
@@
-$EndComp
-$Comp
-L Device:R R3
-U 1 1 6060A7A2
-P 5750 3050
-AR Path="/60607DD9/6060A7A2" Ref="R3"  Part="1"
-AR Path="/60615AFA/6060A7A2" Ref="R?"  Part="1"
-F 0 "R?" H 5820 3096 50  0000 L CNN
-F 1 "33" H 5820 3005 50  0000 L CNN
-F 2 "" V 5680 3050 50  0001 C CNN
-F 3 "~" H 5750 3050 50  0001 C CNN
-	1    5750 3050
-	1    0    0    -1
 $EndComp
 $Comp
@@
 Wire Wire Line
 	6200 3350 6200 3600
-Wire Notes Line
-	5550 2900 6050 2900
-Wire Notes Line
-	6050 2900 6050 3500
-Text Notes 5200 3000 0    50   ~ 0
-Solenoid
-Wire Notes Line
-	5550 3500 5550 2900
-Wire Notes Line
-	6050 3500 5550 3500
 Wire Wire Line
 	5750 3600 5750 3650
-Connection ~ 5750 3600
 Wire Wire Line
 	6200 3600 5750 3600
-Wire Wire Line
-	5750 3500 5750 3600
 Wire Wire Line
 	5400 3850 5450 3850
@@
 F 3 "" H 5750 4250 50  0001 C CNN
 	1    5750 4250
-	1    0    0    -1
-$EndComp
-$Comp
-L Device:L L1
-U 1 1 6060BDB8
-P 5750 3350
-AR Path="/60607DD9/6060BDB8" Ref="L1"  Part="1"
-AR Path="/60615AFA/6060BDB8" Ref="L?"  Part="1"
-F 0 "L?" H 5802 3396 50  0000 L CNN
-F 1 "55mH" H 5802 3305 50  0000 L CNN
-F 2 "" H 5750 3350 50  0001 C CNN
-F 3 "~" H 5750 3350 50  0001 C CNN
-	1    5750 3350
 	1    0    0    -1
 $EndComp
@@
 $EndComp
 Wire Wire Line
-	5750 2750 5750 2900
-Wire Wire Line
 	5750 4050 5750 4250
 Wire Wire Line
 	4900 3850 5000 3850
+Wire Wire Line
+	5750 2750 5750 3600
+Connection ~ 5750 3600
 $EndSCHEMATC

Commit message: add 3.png
Changed lines of the file:
@@
 $Descr A4 11693 8268
 encoding utf-8
-Sheet 3 3
+Sheet 3 4
 Title ""
 Date ""
@@
 $Comp
 L power:+12V #PWR03
-U 1 1 606086E2
+U 1 1 6061936D
 P 6200 2750
-AR Path="/60607DD9/606086E2" Ref="#PWR03"  Part="1"
-AR Path="/60615AFA/606086E2" Ref="#PWR?"  Part="1"
-F 0 "#PWR?" H 6200 2600 50  0001 C CNN
+AR Path="/60607DD9/6061936D" Ref="#PWR03"  Part="1"
+AR Path="/60615AFA/6061936D" Ref="#PWR06"  Part="1"
+F 0 "#PWR06" H 6200 2600 50  0001 C CNN
 F 1 "+12V" H 6215 2923 50  0000 C CNN
 F 2 "" H 6200 2750 50  0001 C CNN
@@
 $Comp
 L Device:R R1
-U 1 1 60609203
+U 1 1 6061936E
 P 5150 3850
-AR Path="/60607DD9/60609203" Ref="R1"  Part="1"
-AR Path="/60615AFA/60609203" Ref="R?"  Part="1"
-F 0 "R?" V 4943 3850 50  0000 C CNN
+AR Path="/60607DD9/6061936E" Ref="R1"  Part="1"
+AR Path="/60615AFA/6061936E" Ref="R4"  Part="1"
+F 0 "R4" V 4943 3850 50  0000 C CNN
 F 1 "100" V 5034 3850 50  0000 C CNN
 F 2 "" V 5080 3850 50  0001 C CNN
@@
 $Comp
 L Device:D D1
-U 1 1 6060B192
+U 1 1 60619371
 P 6200 3200
-AR Path="/60607DD9/6060B192" Ref="D1"  Part="1"
-AR Path="/60615AFA/6060B192" Ref="D?"  Part="1"
-F 0 "D?" V 6154 3280 50  0000 L CNN
+AR Path="/60607DD9/60619371" Ref="D1"  Part="1"
+AR Path="/60615AFA/60619371" Ref="D2"  Part="1"
+F 0 "D2" V 6154 3280 50  0000 L CNN
 F 1 "1N4001/4007" V 6245 3280 50  0000 L CNN
 F 2 "" H 6200 3200 50  0001 C CNN
@@
 $Comp
 L power:GND #PWR01
-U 1 1 6060D913
+U 1 1 60619374
 P 5400 4250
-AR Path="/60607DD9/6060D913" Ref="#PWR01"  Part="1"
-AR Path="/60615AFA/6060D913" Ref="#PWR?"  Part="1"
-F 0 "#PWR?" H 5400 4000 50  0001 C CNN
+AR Path="/60607DD9/60619374" Ref="#PWR01"  Part="1"
+AR Path="/60615AFA/60619374" Ref="#PWR04"  Part="1"
+F 0 "#PWR04" H 5400 4000 50  0001 C CNN
 F 1 "GND" H 5405 4077 50  0000 C CNN
 F 2 "" H 5400 4250 50  0001 C CNN
@@
 $Comp
 L power:GND #PWR02
-U 1 1 6060CB0B
+U 1 1 60619373
 P 5750 4250
-AR Path="/60607DD9/6060CB0B" Ref="#PWR02"  Part="1"
-AR Path="/60615AFA/6060CB0B" Ref="#PWR?"  Part="1"
-F 0 "#PWR?" H 5750 4000 50  0001 C CNN
+AR Path="/60607DD9/60619373" Ref="#PWR02"  Part="1"
+AR Path="/60615AFA/60619373" Ref="#PWR05"  Part="1"
+F 0 "#PWR05" H 5750 4000 50  0001 C CNN
 F 1 "GND" H 5755 4077 50  0000 C CNN
 F 2 "" H 5750 4250 50  0001 C CNN
@@
 $Comp
 L Device:R R2
-U 1 1 6060983D
+U 1 1 6061936F
 P 5400 4050
-AR Path="/60607DD9/6060983D" Ref="R2"  Part="1"
-AR Path="/60615AFA/6060983D" Ref="R?"  Part="1"
-F 0 "R?" H 5470 4096 50  0000 L CNN
+AR Path="/60607DD9/6061936F" Ref="R2"  Part="1"
+AR Path="/60615AFA/6061936F" Ref="R5"  Part="1"
+F 0 "R5" H 5470 4096 50  0000 L CNN
 F 1 "10k" H 5470 4005 50  0000 L CNN
 F 2 "" V 5330 4050 50  0001 C CNN
@@
 $Comp
 L Transistor_FET:BS170 Q1
-U 1 1 60607F3B
+U 1 1 6061936C
 P 5650 3850
-AR Path="/60607DD9/60607F3B" Ref="Q1"  Part="1"
-AR Path="/60615AFA/60607F3B" Ref="Q?"  Part="1"
-F 0 "Q?" H 5854 3896 50  0000 L CNN
+AR Path="/60607DD9/6061936C" Ref="Q1"  Part="1"
+AR Path="/60615AFA/6061936C" Ref="Q2"  Part="1"
+F 0 "Q2" H 5854 3896 50  0000 L CNN
 F 1 "BS170" H 5854 3805 50  0000 L CNN
 F 2 "Package_TO_SOT_THT:TO-92_Inline" H 5850 3775 50  0001 L CIN
