File: analysis/analysis.sch (KiCad schematic (older format))
At the start: 0 parts

Commit message: add 2.png
Changed lines of the file:
@@
 $Descr A4 11693 8268
 encoding utf-8
-Sheet 1 2
+Sheet 1 3
 Title ""
 Date ""
@@
 F1 "Scenario1.sch" 50
 $EndSheet
+$Sheet
+S 1000 2300 2050 750
+U 60615AFA
+F0 "scnario2" 50
+F1 "Scenario2.sch" 50
+$EndSheet
 $EndSCHEMATC

Commit message: add 3.png
Changed lines of the file:
@@
 $Descr A4 11693 8268
 encoding utf-8
-Sheet 1 3
+Sheet 1 4
 Title ""
 Date ""
@@
 F1 "Scenario2.sch" 50
 $EndSheet
+$Sheet
+S 950  3500 2050 750
+U 60616563
+F0 "scenario3" 50
+F1 "Scenario3.sch" 50
+$EndSheet
 $EndSCHEMATC

Commit message: update
Changed lines of the file:
@@
 $Descr A4 11693 8268
 encoding utf-8
-Sheet 1 4
+Sheet 1 5
 Title ""
 Date ""
@@
 F1 "Scenario3.sch" 50
 $EndSheet
+$Sheet
+S 950  4650 2050 750
+U 606051AC
+F0 "scenario4" 50
+F1 "Scenario4.sch" 50
+$EndSheet
 $EndSCHEMATC
